File: palindrome45xt/palindrome40xt3/palindrome40xt3.kicad_sch (KiCad schematic)
At the start: 107 parts, among them Q1 Q_NMOS_GDS, U1 RP2040_Zero

Commit message: upside down version
Parts:
- removed BZ2: Buzzer, TheEndgame2024:Buzzer_Mallory_AST1109MLTRQ, symbol TheEndgame2024:Buzzer
- removed JSOL1: Conn_01x02_Pin, ScottoKeebs_Components:Connector_1x02_JST-PH, symbol Connector:Conn_01x02_Pin
- added JSOL1: Conn_01x02_MountingPin, symbol Connector_Generic_MountingPin:Conn_01x02_MountingPin
Connections:
- net +5V_SOL: now also JSOL1.1 (Pin_1)
- net COIL_LOW: now also JSOL1.2 (Pin_2)
- net GND: now also JSOL1.MP (MountPin)
Changed lines of the file:
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@@
 	)
 	(rectangle
-		(start 229.87 80.01)
+		(start 204.47 69.85)
 		(end 251.46 90.17)
 		(stroke
@@
 	(text "mm yummy buzzer\n"
 		(exclude_from_sim no)
-		(at 240.538 77.978 0)
+		(at 227.584 68.58 0)
 		(effects
 			(font
@@
 	(wire
 		(pts
+			(xy 204.47 140.97) (xy 203.2 140.97)
+		)
+		(stroke
+			(width 0)
+			(type default)
+		)
+	)
+	(wire
+		(pts
 			(xy 127 119.38) (xy 127 138.43)
 		)
@@
 	)
 	(label "COIL_LOW"
-		(at 207.01 129.54 0)
+		(at 234.95 113.03 0)
 		(fields_autoplaced yes)
 		(effects
@@
 		)
 		(property "COIL_LOW" ""
-			(at 207.01 130.81 0)
+			(at 234.95 114.3 0)
 			(effects
 				(font
@@
 	)
 	(label "COIL_LOW"
-		(at 234.95 113.03 0)
+		(at 198.12 135.89 180)
 		(fields_autoplaced yes)
 		(effects
@@
 				(size 1.27 1.27)
 			)
-			(justify left bottom)
+			(justify right bottom)
 		)
 		(property "COIL_LOW" ""
-			(at 234.95 114.3 0)
+			(at 198.12 137.16 0)
+			(effects
+				(font
+					(size 1.27 1.27)
+					(italic yes)
+				)
+				(justify right)
+			)
+		)
+	)
+	(label "GND"
+		(at 204.47 140.97 0)
+		(fields_autoplaced yes)
+		(effects
+			(font
+				(size 1.27 1.27)
+			)
+			(justify left bottom)
+		)
+		(property "GND" ""
+			(at 204.47 142.24 0)
 			(effects
 				(font
@@
 		)
 	)
-	(label "GND"
-		(at 223.52 160.02 0)
+	(label "+5V_SOL"
+		(at 198.12 133.35 180)
 		(fields_autoplaced yes)
 		(effects
@@
 				(size 1.27 1.27)
 			)
-			(justify left bottom)
+			(justify right bottom)
 		)
-		(property "GND" ""
-			(at 223.52 161.29 0)
+		(property "+12V_SOL" ""
+			(at 198.12 134.62 0)
 			(effects
 				(font
@@
 					(italic yes)
 				)
-				(justify left)
+				(justify right)
 			)
 		)
 	)
-	(label "+5V_SOL"
-		(at 207.01 127 0)
+	(label "GND"
+		(at 223.52 160.02 0)
 		(fields_autoplaced yes)
 		(effects
@@
 			(justify left bottom)
 		)
-		(property "+12V_SOL" ""
-			(at 207.01 128.27 0)
+		(property "GND" ""
+			(at 223.52 161.29 0)
 			(effects
 				(font
@@
 		)
 	)
-	(global_label "Sound"
-		(shape input)
-		(at 238.76 82.55 180)
-		(fields_autoplaced yes)
-		(effects
-			(font
-				(size 1.27 1.27)
-			)
-			(justify right)
-		)
-		(property "Intersheetrefs" "${INTERSHEET_REFS}"
-			(at 230.0487 82.55 0)
-			(effects
-				(font
-					(size 1.27 1.27)
-				)
-				(justify right)
-				(hide yes)
-			)
-		)
-	)
 	(global_label "row3"
 		(shape input)
@@
 		)
 	)
-	(global_label "gnd"
-		(shape input)
-		(at 238.76 87.63 180)
-		(fields_autoplaced yes)
-		(effects
-			(font
-				(size 1.27 1.27)
-			)
-			(justify right)
-		)
-		(property "Intersheetrefs" "${INTERSHEET_REFS}"
-			(at 232.3278 87.63 0)
-			(effects
-				(font
-					(size 1.27 1.27)
-				)
-				(justify right)
-				(hide yes)
-			)
-		)
-	)
 	(global_label "row1"
 		(shape input)
@@
 	)
 	(symbol
-		(lib_id "Connector:Conn_01x02_Pin")
-		(at 201.93 127 0)
-		(unit 1)
-		(exclude_from_sim no)
-		(in_bom yes)
-		(on_board yes)
-		(dnp no)
-		(fields_autoplaced yes)
-		(property "Reference" "JSOL1"
-			(at 202.565 121.92 0)
-			(effects
-				(font
-					(size 1.27 1.27)
-				)
-			)
-		)
-		(property "Value" "Conn_01x02_Pin"
-			(at 202.565 124.46 0)
-			(effects
-				(font
-					(size 1.27 1.27)
-				)
-			)
-		)
-		(property "Footprint" "ScottoKeebs_Components:Connector_1x02_JST-PH"
-			(at 201.93 127 0)
-			(effects
-				(font
-					(size 1.27 1.27)
-				)
-				(hide yes)
-			)
-		)
-		(property "Datasheet" "~"
-			(at 201.93 127 0)
-			(effects
-				(font
-					(size 1.27 1.27)
-				)
-				(hide yes)
-			)
-		)
-		(property "Description" "Generic connector, single row, 01x02, script generated"
-			(at 201.93 127 0)
-			(effects
-				(font
-					(size 1.27 1.27)
-				)
-				(hide yes)
-			)
-		)
-		(pin "2"
-		)
-		(pin "1"
-		)
-		(instances
-			(project ""
-				(path "/5b67e7e4-7b9c-457b-a2d8-b25d5b0c8cf3"
-					(reference "JSOL1")
-					(unit 1)
-				)
-			)
-		)
-	)
-	(symbol
 		(lib_id "ScottoKeebs:Placeholder_Keyswitch")
 		(at 119.38 121.92 0)
@@
 	)
 	(symbol
+		(lib_id "Connector_Generic_MountingPin:Conn_01x02_MountingPin")
+		(at 203.2 133.35 0)
+		(unit 1)
+		(exclude_from_sim no)
+		(in_bom yes)
+		(on_board yes)
+		(dnp no)
+		(fields_autoplaced yes)
+		(property "Reference" "JSOL1"
+			(at 205.74 133.7056 0)
+			(effects
+				(font
+					(size 1.27 1.27)
+				)
+				(justify left)
+			)
+		)
+		(property "Value" "Conn_01x02_MountingPin"
+			(at 205.74 136.2456 0)
+			(effects
+				(font
+					(size 1.27 1.27)
+				)
+				(justify left)
+			)
+		)
+		(property "Footprint" ""
+			(at 203.2 133.35 0)
+			(effects
+				(font
+					(size 1.27 1.27)
+				)
+				(hide yes)
+			)
+		)
+		(property "Datasheet" "~"
+			(at 203.2 133.35 0)
+			(effects
+				(font
+					(size 1.27 1.27)
+				)
+				(hide yes)
+			)
+		)
+		(property "Description" "Generic connectable mounting pin connector, single row, 01x02, script generated (kicad-library-utils/schlib/autogen/connector/)"
+			(at 203.2 133.35 0)
+			(effects
+				(font
+					(size 1.27 1.27)
+				)
+				(hide yes)
+			)
+		)
+		(pin "MP"
+		)
+		(pin "2"
+		)
+		(pin "1"
+		)
+		(instances
+			(project ""
+				(path "/5b67e7e4-7b9c-457b-a2d8-b25d5b0c8cf3"
+					(reference "JSOL1")
+					(unit 1)
+				)
+			)
+		)
+	)
+	(symbol
 		(lib_id "ScottoKeebs:Placeholder_Keyswitch")
 		(at 129.54 82.55 0)
@@
 					(unit 1)
 				)
-			)
-		)
-	)
-	(symbol
-		(lib_id "TheEndgame2024:Buzzer")
-		(at 241.3 85.09 0)
-		(unit 1)
-		(exclude_from_sim no)
-		(in_bom yes)
-		(on_board yes)
-		(dnp no)
-		(fields_autoplaced yes)
-		(property "Reference" "BZ2"
-			(at 245.11 84.455 0)
-			(effects
-				(font
-					(size 1.27 1.27)
-				)
-				(justify left)
-			)
-		)
-		(property "Value" "Buzzer"
-			(at 245.11 86.995 0)
-			(effects
-				(font
-					(size 1.27 1.27)
-				)
-				(justify left)
-			)
-		)
-		(property "Footprint" "TheEndgame2024:Buzzer_Mallory_AST1109MLTRQ"
-			(at 240.665 82.55 90)
-			(effects
-				(font
-					(size 1.27 1.27)
-				)
-				(hide yes)
-			)
-		)
-		(property "Datasheet" "~"
-			(at 240.665 82.55 90)
-			(effects
-				(font
-					(size 1.27 1.27)
-				)
-				(hide yes)
-			)
-		)
-		(property "Description" ""
-			(at 241.3 85.09 0)
-			(effects
-				(font
-					(size 1.27 1.27)
-				)
-				(hide yes)
-			)
-		)
-		(pin "1"
-		)
-		(pin "2"
-		)
-		(instances
-			(project "palindrome45xt2"
-				(path "/5b67e7e4-7b9c-457b-a2d8-b25d5b0c8cf3"
-					(reference "BZ2")
-					(unit 1)
-				)

Commit message: almost done
Parts:
- removed H1: M3 GND BOLT, MountingHole:MountingHole_3.2mm_M3_Pad, symbol Mechanical:MountingHole_Pad
- JSOL1: footprint (none) -> Connector_JST:JST_SH_SM02B-SRSS-TB_1x02-1MP_P1.00mm_Horizontal
Connections:
- net col0: now also U1.3 (2); no longer U1.20 (29)
- net col1: now also U1.4 (3); no longer U1.19 (28)
- net col10: now also U1.17 (26); no longer U1.6 (5)
- net col11: now also U1.18 (27); no longer U1.5 (4)
- net col12: now also U1.19 (28); no longer U1.4 (3)
- net col13: now also U1.20 (29); no longer U1.3 (2)
- net col2: now also U1.5 (4); no longer U1.18 (27)
- net col3: now also U1.6 (5); no longer U1.17 (26)
- net col4: now also U1.7 (6); no longer U1.16 (15)
- net col5: now also U1.8 (7); no longer U1.15 (14)
- net col6: now also U1.9 (8); no longer U1.14 (13)
- net col7: now also U1.14 (13); no longer U1.10 (9)
- net col8: now also U1.15 (14); no longer U1.8 (7)
- net col9: now also U1.16 (15); no longer U1.7 (6)
- net row0: now also U1.10 (9); no longer U1.9 (8)
- net row1: now also U1.13 (12); no longer U1.11 (10)
- net row3: now also U1.11 (10); no longer U1.13 (12)
- no-connect marks 0 -> 2
Other:
- moved on the sheet: U1
