File: palindrome45xt/palindrome40xt3/palindrome40xt3.kicad_sch (KiCad schematic)
At the start: 110 parts, among them J1 Conn_01x02_Socket, Q1 Q_NMOS_GDS, Q3 TIP120, U1 RP2040_Zero

Commit message: ww
Parts:
- removed D52: 1N4004, ergodonk_simple_zero:D_DO-41_SOD81_P10.16mm_Horizontal, symbol Diode:1N4004
- removed J1: Conn_01x02_Socket, ergodonk_simple_zero:PinHeader_1x02_P2.54mm_Vertical, symbol Connector:Conn_01x02_Socket
- removed J_SOL_1: Conn_01x02_Female, ergodonk_simple_zero:PinHeader_1x02_P2.54mm_Vertical, symbol Connector:Conn_01x02_Socket
- removed Q3: TIP120, ergodonk_simple_zero:TO-220-3_Horizontal_TabDown_ergodonk_simple_zero, symbol Transistor_BJT:TIP120
- removed R4: 1k, ergodonk_simple_zero:R_Axial_DIN0309_L9.0mm_D3.2mm_P12.70mm_Horizontal, symbol Device:R_Small
Connections:
- no-connect marks 6 -> 2
Other:
- note removed: "Alternate Solenoid socket for short wires"

Commit message: pre disaster
Parts:
- added H1: M3 GND BOLT, MountingHole:MountingHole_3.2mm_M3_Pad, symbol Mechanical:MountingHole_Pad
Connections:
- net GND: now also H1.1
Changed lines of the file:
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@@
 		)
 	)
+	(label "GND"
+		(at 256.54 144.78 180)
+		(fields_autoplaced yes)
+		(effects
+			(font
+				(size 1.27 1.27)
+			)
+			(justify right bottom)
+		)
+		(property "GND" ""
+			(at 256.54 146.05 0)
+			(effects
+				(font
+					(size 1.27 1.27)
+					(italic yes)
+				)
+				(justify right)
+			)
+		)
+	)
 	(label "COIL_LOW"
 		(at 231.14 140.97 0)
@@
 					(unit 1)
 				)
+			)
+		)
+	)
+	(symbol
+		(lib_id "Mechanical:MountingHole_Pad")
+		(at 256.54 142.24 0)
+		(unit 1)
+		(exclude_from_sim no)
+		(in_bom no)
+		(on_board yes)
+		(dnp no)
+		(fields_autoplaced yes)
+		(property "Reference" "H1"
+			(at 259.08 139.7 0)
+			(effects
+				(font
+					(size 1.27 1.27)
+				)
+				(justify left)
+			)
+		)
+		(property "Value" "M3 GND BOLT"
+			(at 259.08 142.24 0)
+			(effects
+				(font
+					(size 1.27 1.27)
+				)
+				(justify left)
+			)
+		)
+		(property "Footprint" "MountingHole:MountingHole_3.2mm_M3_Pad"
+			(at 256.54 142.24 0)
+			(effects
+				(font
+					(size 1.27 1.27)
+				)
+				(hide yes)
+			)
+		)
+		(property "Datasheet" "~"
+			(at 256.54 142.24 0)
+			(effects
+				(font
+					(size 1.27 1.27)
+				)
+				(hide yes)
+			)
+		)
+		(property "Description" "Mounting Hole with connection"
+			(at 256.54 142.24 0)
+			(effects
+				(font
+					(size 1.27 1.27)
+				)
+				(hide yes)
+			)
+		)
+		(pin "1"
+		)
+		(instances
+			(project "palindrome40xt3"
+				(path "/5b67e7e4-7b9c-457b-a2d8-b25d5b0c8cf3"
+					(reference "H1")
+					(unit 1)
+				)
