File: palindrome45xt/palindrome40xt3/palindrome40xt3.kicad_sch (KiCad schematic)
At the start: 110 parts, among them J1 Conn_01x02_Socket, Q1 Q_NMOS_GDS, Q3 TIP120, U1 RP2040_Zero

Commit message: disaster here
Parts:
- removed C1: 0.1uF, Capacitor_SMD:C_0805_2012Metric, symbol Device:C
- removed D51: D_Schottky, Diode_SMD:D_SOD-123, symbol Device:D_Schottky
- removed JSOL1: Conn_01x02_MountingPin, Connector_JST:JST_SH_SM02B-SRSS-TB_1x02-1MP_P1.00mm_Horizontal, symbol Connector_Generic_MountingPin:Conn_01x02_MountingPin
- removed Q1: Q_NMOS_GDS, Package_TO_SOT_THT:TO-220-3_Horizontal_TabDown, symbol Transistor_FET:Q_NMOS_GDS
- removed R1: 100, Resistor_SMD:R_0805_2012Metric, symbol Device:R
- removed R2: 100k, Resistor_SMD:R_0805_2012Metric, symbol Device:R
Connections:
- no-connect marks 6 -> 2
Other:
- note removed: "SOLENOID SUPPORT WOOO"
- moved on the sheet: D52, J1, J_SOL_1, Q3, R4

Commit message: rewiring time
Parts:
- removed R4: 1k, ergodonk_simple_zero:R_Axial_DIN0309_L9.0mm_D3.2mm_P12.70mm_Horizontal, symbol Device:R_Small
- added R1: 1k, Resistor_THT:R_Axial_DIN0309_L9.0mm_D3.2mm_P12.70mm_Horizontal, symbol Device:R_Small
Connections:
- net SOLENOID_EN: now also R1.1
- net at Q3.1 (B): now also R1.2
Changed lines of the file:
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@@
 	(wire
 		(pts
-			(xy 96.52 50.8) (xy 92.71 50.8)
+			(xy 97.79 50.8) (xy 92.71 50.8)
 		)
 		(stroke
@@
 	(wire
 		(pts
-			(xy 101.6 50.8) (xy 105.41 50.8)
+			(xy 102.87 50.8) (xy 105.41 50.8)
 		)
 		(stroke
@@
 	)
 	(symbol
+		(lib_id "Device:R_Small")
+		(at 100.33 50.8 90)
+		(unit 1)
+		(exclude_from_sim no)
+		(in_bom yes)
+		(on_board yes)
+		(dnp no)
+		(fields_autoplaced yes)
+		(property "Reference" "R1"
+			(at 100.33 45.72 90)
+			(effects
+				(font
+					(size 1.016 1.016)
+				)
+			)
+		)
+		(property "Value" "1k"
+			(at 100.33 48.26 90)
+			(effects
+				(font
+					(size 1.27 1.27)
+				)
+			)
+		)
+		(property "Footprint" "Resistor_THT:R_Axial_DIN0309_L9.0mm_D3.2mm_P12.70mm_Horizontal"
+			(at 100.33 50.8 0)
+			(effects
+				(font
+					(size 1.27 1.27)
+				)
+				(hide yes)
+			)
+		)
+		(property "Datasheet" "~"
+			(at 100.33 50.8 0)
+			(effects
+				(font
+					(size 1.27 1.27)
+				)
+				(hide yes)
+			)
+		)
+		(property "Description" "Resistor, small symbol"
+			(at 100.33 50.8 0)
+			(effects
+				(font
+					(size 1.27 1.27)
+				)
+				(hide yes)
+			)
+		)
+		(pin "1"
+		)
+		(pin "2"
+		)
+		(instances
+			(project ""
+				(path "/5b67e7e4-7b9c-457b-a2d8-b25d5b0c8cf3"
+					(reference "R1")
+					(unit 1)
+				)
+			)
+		)
+	)
+	(symbol
 		(lib_id "ScottoKeebs:Placeholder_Diode")
 		(at 111.76 109.22 90)
@@
 					(unit 1)
 				)
-			)
-		)
-	)
-	(symbol
-		(lib_name "R_Small_1")
-		(lib_id "Device:R_Small")
-		(at 99.06 50.8 90)
-		(unit 1)
-		(exclude_from_sim no)
-		(in_bom yes)
-		(on_board yes)
-		(dnp no)
-		(fields_autoplaced yes)
-		(property "Reference" "R4"
-			(at 99.06 45.72 90)
-			(effects
-				(font
-					(size 1.016 1.016)
-				)
-			)
-		)
-		(property "Value" "1k"
-			(at 99.06 48.26 90)
-			(effects
-				(font
-					(size 1.27 1.27)
-				)
-			)
-		)
-		(property "Footprint" "ergodonk_simple_zero:R_Axial_DIN0309_L9.0mm_D3.2mm_P12.70mm_Horizontal"
-			(at 99.06 50.8 0)
-			(effects
-				(font
-					(size 1.27 1.27)
-				)
-				(hide yes)
-			)
-		)
-		(property "Datasheet" "~"
-			(at 99.06 50.8 0)
-			(effects
-				(font
-					(size 1.27 1.27)
-				)
-				(hide yes)
-			)
-		)
-		(property "Description" "Resistor, small symbol"
-			(at 99.06 50.8 0)
-			(effects
-				(font
-					(size 1.27 1.27)
-				)
-				(hide yes)
-			)
-		)
-		(pin "1"
-		)
-		(pin "2"
-		)
-		(instances
-			(project ""
-				(path "/5b67e7e4-7b9c-457b-a2d8-b25d5b0c8cf3"
-					(reference "R4")
-					(unit 1)
-				)

Commit message: donezo
Parts:
- removed D8: Diode, Diode_SMD:D_SOD-123, symbol ScottoKeebs:Placeholder_Diode
- removed J1: Conn_01x02_Socket, ergodonk_simple_zero:PinHeader_1x02_P2.54mm_Vertical, symbol Connector:Conn_01x02_Socket
Connections:
- net Y_KEY: now reaches S8.2
- net Y_KEY: now also U1.2 (1)
- no-connect marks 2 -> 1
Other:
- moved on the sheet: S8
Changed lines of the file:
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@@
 	)
 	(junction
-		(at 102.87 41.91)
-		(diameter 0)
-		(color 0 0 0 0)
-	)
-	(junction
 		(at 142.24 113.03)
 		(diameter 0)
@@
 	)
 	(junction
-		(at 102.87 31.75)
-		(diameter 0)
-		(color 0 0 0 0)
-	)
-	(junction
 		(at 76.2 80.01)
 		(diameter 0)
@@
 	)
 	(junction
-		(at 101.6 92.71)
-		(diameter 0)
-		(color 0 0 0 0)
-	)
-	(junction
 		(at 25.4 113.03)
 		(diameter 0)
@@
 	)
 	(junction
+		(at 96.52 80.01)
+		(diameter 0)
+		(color 0 0 0 0)
+	)
+	(junction
 		(at 127 80.01)
 		(diameter 0)
@@
 	)
 	(junction
-		(at 96.52 80.01)
-		(diameter 0)
-		(color 0 0 0 0)
-	)
-	(junction
 		(at 142.24 92.71)
 		(diameter 0)
@@
 		(at 210.82 38.1)
 	)
-	(no_connect
-		(at 185.42 35.56)
-	)
 	(wire
 		(pts
@@
 	(wire
 		(pts
-			(xy 96.52 80.01) (xy 96.52 100.33)
+			(xy 81.28 132.08) (xy 91.44 132.08)
 		)
 		(stroke
@@
 	(wire
 		(pts
-			(xy 81.28 132.08) (xy 91.44 132.08)
+			(xy 96.52 72.39) (xy 96.52 80.01)
 		)
 		(stroke
@@
 	(wire
 		(pts
-			(xy 102.87 41.91) (xy 102.87 39.37)
-		)
-		(stroke
-			(width 0)
-			(type default)
-		)
-	)
-	(wire
-		(pts
 			(xy 71.12 113.03) (xy 81.28 113.03)
 		)
@@
 	(wire
 		(pts
-			(xy 111.76 92.71) (xy 121.92 92.71)
+			(xy 96.52 80.01) (xy 97.79 80.01)
 		)
 		(stroke
@@
 	(wire
 		(pts
-			(xy 83.82 39.37) (xy 83.82 41.91)
+			(xy 111.76 92.71) (xy 121.92 92.71)
 		)
 		(stroke
@@
 	(wire
 		(pts
-			(xy 101.6 92.71) (xy 111.76 92.71)
-		)
-		(stroke
-			(width 0)
-			(type default)
-		)
-	)
-	(wire
-		(pts
 			(xy 60.96 113.03) (xy 71.12 113.03)
 		)
@@
 	(wire
 		(pts
-			(xy 96.52 72.39) (xy 96.52 80.01)
+			(xy 91.44 92.71) (xy 111.76 92.71)
 		)
 		(stroke
@@
 	(wire
 		(pts
-			(xy 83.82 41.91) (xy 102.87 41.91)
-		)
-		(stroke
-			(width 0)
-			(type default)
-		)
-	)
-	(wire
-		(pts
 			(xy 113.03 30.48) (xy 113.03 31.75)
 		)
@@
 	(wire
 		(pts
-			(xy 102.87 43.18) (xy 102.87 41.91)
+			(xy 102.87 39.37) (xy 102.87 43.18)
 		)
 		(stroke
@@
 	(wire
 		(pts
-			(xy 91.44 92.71) (xy 101.6 92.71)
-		)
-		(stroke
-			(width 0)
-			(type default)
-		)
-	)
-	(wire
-		(pts
-			(xy 83.82 36.83) (xy 83.82 31.75)
-		)
-		(stroke
-			(width 0)
-			(type default)
-		)
-	)
-	(wire
-		(pts
 			(xy 86.36 80.01) (xy 86.36 100.33)
 		)
@@
 	(wire
 		(pts
-			(xy 83.82 31.75) (xy 102.87 31.75)
-		)
-		(stroke
-			(width 0)
-			(type default)
-		)
-	)
-	(wire
-		(pts
 			(xy 91.44 113.03) (xy 101.6 113.03)
 		)
@@
 	(wire
 		(pts
+			(xy 96.52 80.01) (xy 96.52 100.33)
+		)
+		(stroke
+			(width 0)
+			(type default)
+		)
+	)
+	(wire
+		(pts
 			(xy 113.03 43.18) (xy 113.03 45.72)
 		)
@@
 		)
 	)
+	(global_label "Y_KEY"
+		(shape input)
+		(at 102.87 85.09 270)
+		(fields_autoplaced yes)
+		(effects
+			(font
+				(size 1.27 1.27)
+			)
+			(justify right)
+		)
+		(property "Intersheetrefs" "${INTERSHEET_REFS}"
+			(at 102.87 92.6917 90)
+			(effects
+				(font
+					(size 1.27 1.27)
+				)
+				(justify right)
+				(hide yes)
+			)
+		)
+	)
 	(global_label "col6"
 		(shape input)
@@
 		)
 	)
+	(global_label "Y_KEY"
+		(shape input)
+		(at 185.42 35.56 180)
+		(fields_autoplaced yes)
+		(effects
+			(font
+				(size 1.27 1.27)
+			)
+			(justify right)
+		)
+		(property "Intersheetrefs" "${INTERSHEET_REFS}"
+			(at 177.8183 35.56 0)
+			(effects
+				(font
+					(size 1.27 1.27)
+				)
+				(justify right)
+				(hide yes)
+			)
+		)
+	)
 	(global_label "col9"
 		(shape input)
@@
 	(symbol
 		(lib_id "ScottoKeebs:Placeholder_Keyswitch")
-		(at 99.06 82.55 0)
+		(at 100.33 82.55 0)
 		(unit 1)
 		(exclude_from_sim no)
@@
 		(on_board yes)
 		(dnp no)
-		(fields_autoplaced yes)
 		(property "Reference" "S8"
-			(at 99.06 74.93 0)
+			(at 100.33 74.93 0)
 			(effects
 				(font
@@
 		)
 		(property "Value" "Y"
-			(at 99.06 77.47 0)
+			(at 100.33 77.47 0)
 			(effects
 				(font
@@
 		)
 		(property "Footprint" "Button_Switch_Keyboard:SW_Cherry_MX_1.00u_PCB"
-			(at 99.06 82.55 0)
+			(at 100.33 82.55 0)
 			(effects
 				(font
@@
 		)
 		(property "Datasheet" "~"
-			(at 99.06 82.55 0)
+			(at 100.33 82.55 0)
 			(effects
 				(font
@@
 		)
 		(property "Description" "Push button switch, normally open, two pins, 45° tilted"
-			(at 99.06 82.55 0)
+			(at 100.33 82.55 0)
 			(effects
 				(font
@@
 	)
 	(symbol
-		(lib_id "ScottoKeebs:Placeholder_Diode")
-		(at 101.6 88.9 90)
-		(unit 1)
-		(exclude_from_sim no)
-		(in_bom yes)
-		(on_board yes)
-		(dnp no)
-		(fields_autoplaced yes)
-		(property "Reference" "D8"
-			(at 104.14 87.63 90)
-			(effects
-				(font
-					(size 1.27 1.27)
-				)
-				(justify right)
-			)
-		)
-		(property "Value" "Diode"
-			(at 104.14 90.17 90)
-			(effects
-				(font
-					(size 1.27 1.27)
-				)
-				(justify right)
-			)
-		)
-		(property "Footprint" "Diode_SMD:D_SOD-123"
-			(at 101.6 88.9 0)
-			(effects
-				(font
-					(size 1.27 1.27)
-				)
-				(hide yes)
-			)
-		)
-		(property "Datasheet" ""
-			(at 101.6 88.9 0)
-			(effects
-				(font
-					(size 1.27 1.27)
-				)
-				(hide yes)
-			)
-		)
-		(property "Description" "1N4148 (DO-35) or 1N4148W (SOD-123)"
-			(at 101.6 88.9 0)
-			(effects
-				(font
-					(size 1.27 1.27)
-				)
-				(hide yes)
-			)
-		)
-		(property "Sim.Device" "D"
-			(at 101.6 88.9 0)
-			(effects
-				(font
-					(size 1.27 1.27)
-				)
-				(hide yes)
-			)
-		)
-		(property "Sim.Pins" "1=K 2=A"
-			(at 101.6 88.9 0)
-			(effects
-				(font
-					(size 1.27 1.27)
-				)
-				(hide yes)
-			)
-		)
-		(pin "1"
-		)
-		(pin "2"
-		)
-		(instances
-			(project "palindrome45xt"
-				(path "/5b67e7e4-7b9c-457b-a2d8-b25d5b0c8cf3"
-					(reference "D8")
-					(unit 1)
-				)
-			)
-		)
-	)
-	(symbol
 		(lib_id "ScottoKeebs:MCU_RP2040_Zero")
 		(at 198.12 41.91 0)
@@
 					(unit 1)
 				)
-			)
-		)
-	)
-	(symbol
-		(lib_id "Connector:Conn_01x02_Socket")
-		(at 78.74 39.37 180)
-		(unit 1)
-		(exclude_from_sim no)
-		(in_bom yes)
-		(on_board yes)
-		(dnp no)
-		(fields_autoplaced yes)
-		(property "Reference" "J1"
-			(at 79.375 31.75 0)
-			(effects
-				(font
-					(size 1.27 1.27)
-				)
-			)
-		)
-		(property "Value" "Conn_01x02_Socket"
-			(at 79.375 34.29 0)
-			(effects
-				(font
-					(size 1.27 1.27)
-				)
-			)
-		)
-		(property "Footprint" "ergodonk_simple_zero:PinHeader_1x02_P2.54mm_Vertical"
-			(at 78.74 39.37 0)
-			(effects
-				(font
-					(size 1.27 1.27)
-				)
-				(hide yes)
-			)
-		)
-		(property "Datasheet" "~"
-			(at 78.74 39.37 0)
-			(effects
-				(font
-					(size 1.27 1.27)
-				)
-				(hide yes)
-			)
-		)
-		(property "Description" "Generic connector, single row, 01x02, script generated"
-			(at 78.74 39.37 0)
-			(effects
-				(font
-					(size 1.27 1.27)
-				)
-				(hide yes)
-			)
-		)
-		(pin "1"
-		)
-		(pin "2"
-		)
-		(instances
-			(project ""
-				(path "/5b67e7e4-7b9c-457b-a2d8-b25d5b0c8cf3"
-					(reference "J1")
-					(unit 1)
-				)
