File: palindrome45xt/palindrome40xt3/palindrome40xt3.kicad_pcb (KiCad board)
At the start: 2 copper layers, 295.8 x 87 mm, 110 parts, among them J1 Conn_01x02_Socket, Q1 Q_NMOS_GDS, Q3 TIP120, U1 RP2040_Zero

Commit message: ww
Parts:
- removed D52: 1N4004, ergodonk_simple_zero:D_DO-41_SOD81_P10.16mm_Horizontal
- removed J1: Conn_01x02_Socket, ergodonk_simple_zero:PinHeader_1x02_P2.54mm_Vertical
- removed J_SOL_1: Conn_01x02_Female, ergodonk_simple_zero:PinHeader_1x02_P2.54mm_Vertical
- removed Q3: TIP120, ergodonk_simple_zero:TO-220-3_Horizontal_TabDown_ergodonk_simple_zero
- removed R4: 1k, ergodonk_simple_zero:R_Axial_DIN0309_L9.0mm_D3.2mm_P12.70mm_Horizontal
- moved D27 80.0 mm to (319.3, 131.8)
- moved D30 80.0 mm to (109.8, 150.9)
- moved D31 80.0 mm to (136.0, 150.9)
- moved D32 80.0 mm to (155.0, 150.9)
- moved D37 80.0 mm to (250.3, 150.9)
- moved D39 80.0 mm to (288.4, 150.9)
- moved D49 80.0 mm to (307.4, 169.9)
- moved S32 80.0 mm to (149.9, 147.8)
- moved S33 80.0 mm to (169.0, 147.8)
- moved S35 80.0 mm to (207.1, 147.8)
- moved S38 80.0 mm to (264.2, 147.8)
- moved S39 80.0 mm to (283.3, 147.8)
- moved D1 80.0 mm to (78.8, 112.8)
- moved D14 80.0 mm to (345.6, 112.6)
- moved D15 80.0 mm to (78.8, 131.8)
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Routing:
- net /GND: track 322.4 -> 324.5 mm
- added copper zone on B.Cu, net (none)
- added copper zone on F.Cu, net (none)
Other:
- board size 295.8 x 87 mm -> 295.8 x 84.1 mm
- board text added: "Tighty40"
- board text added: "Whitey40"
