File: palindrome45xt/palindrome40xt3/palindrome40xt3.kicad_pcb (KiCad board)
At the start: 2 copper layers, 295.9 x 82.9 mm, 100 parts, among them U1 RP2040_Zero

Commit message: upside down version
Parts:
- removed H1: M3 GND BOLT, MountingHole:MountingHole_3.2mm_M3_Pad
- added C1: 0.1uF, Capacitor_SMD:C_0805_2012Metric, F.Cu at (159.5, 96.0)
- added D51: D_Schottky, Diode_SMD:D_SOD-123, F.Cu at (160.0, 89.5)
- added JSOL1: Conn_01x02_MountingPin, Connector_JST:JST_SH_BM02B-SRSS-TB_1x02-1MP_P1.00mm_Vertical, B.Cu at (150.5, 32.0)
- added Q1: Q_NMOS_GDS, Package_TO_SOT_THT:TO-220-3_Horizontal_TabDown, F.Cu at (169.5, 92.3)
- added R1: 100, Resistor_SMD:R_0805_2012Metric, F.Cu at (174.0, 92.0)
- added R2: 100k, Resistor_SMD:R_0805_2012Metric, B.Cu at (167.0, 98.5)
- moved D34 12.4 mm to (146.5, 85.0)
- moved D6 12.2 mm to (132.5, 47.0)
- moved D22 1.58 mm to (178.0, 67.5)
Connections:
- U1 pad 10: row1 -> col7
- U1 pad 11: row2 -> row1
- U1 pad 12: row3 -> row2
- U1 pad 13: col7 -> row3
- U1 pad 22: GND -> /GND
Routing:
- net /SOLENOID_EN: track 0.00 -> 123.0 mm, vias 0 -> 2
- net /GND: track 0.00 -> 108.0 mm, vias 0 -> 3
- net /+5V_SOL: track 0.00 -> 90.5 mm, vias 0 -> 1
- net /COIL_LOW: track 0.00 -> 89.0 mm, vias 0 -> 2
- net row3: track 214.4 -> 286.3 mm, vias 0 -> 4
- net row2: track 315.6 -> 368.9 mm, vias 0 -> 2
- net row1: track 313.8 -> 350.7 mm
- net Net-(Q1-G): track 0.00 -> 10.6 mm
- net Net-(D34-A): track 11.9 -> 4.80 mm
- net Net-(D6-A): track 11.9 -> 5.02 mm
- net Net-(D7-A): track 0.00 -> 5.49 mm
- net row0: track 397.1 -> 391.9 mm
- net col11: track 146.5 -> 150.6 mm
- net Net-(D22-A): track 7.53 -> 9.32 mm
- net col7: track 65.6 -> 66.9 mm
Other:
- board size 295.9 x 82.9 mm -> 295.9 x 87 mm

Commit message: almost done
Parts:
- C1, D51, Q1, R1, U1: moved to B.Cu
- D41: moved to F.Cu
- JSOL1: footprint Connector_JST:JST_SH_BM02B-SRSS-TB_1x02-1MP_P1.00mm_Vertical -> Connector_JST:JST_SH_SM02B-SRSS-TB_1x02-1MP_P1.00mm_Horizontal
- moved C1 16.1 mm to (173.5, 88.0), turned to -90 degrees
- moved D51 13.6 mm to (173.0, 93.5), turned to -90 degrees
- moved R1 11.7 mm to (164.0, 86.0), turned to -90 degrees
- moved R2 9.55 mm to (160.5, 91.5), turned to 90 degrees
- moved JSOL1 7.66 mm to (145.5, 37.8), turned to 90 degrees
- moved Q1 5.58 mm to (164.0, 92.3), turned to 0 degrees
- moved D41 0.30 mm to (310.0, 79.5)
- turned U1 to 180 degrees
Connections:
- U1 pad 10: col7 -> row0
- U1 pad 11: row1 -> row3
- U1 pad 13: row3 -> row1
- U1 pad 14: col6 -> col7
- U1 pad 15: col5 -> col8
- U1 pad 16: col4 -> col9
- U1 pad 17: col3 -> col10
- U1 pad 18: col2 -> col11
- U1 pad 19: col1 -> col12
- U1 pad 20: col0 -> col13
- U1 pad 3: col13 -> col0
- U1 pad 4: col12 -> col1
- U1 pad 5: col11 -> col2
- U1 pad 6: col10 -> col3
- U1 pad 7: col9 -> col4
- U1 pad 8: col8 -> col5
- U1 pad 9: row0 -> col6
Routing:
- net /+5V_SOL: track 90.5 -> 197.3 mm, vias 1 -> 4
- net /GND: track 108.0 -> 200.1 mm, vias 3 -> 4
- net /SOLENOID_EN: track 123.0 -> 74.9 mm
- net /COIL_LOW: track 89.0 -> 72.2 mm, vias 2 -> 1
- net Net-(D47-A): track 0.00 -> 11.9 mm
- net Net-(D41-A): track 11.9 -> 0.00 mm
- net Net-(Q1-G): track 10.6 -> 14.8 mm
- net col2: track 157.1 -> 153.2 mm
- net col3: track 139.9 -> 136.0 mm
- net col4: track 103.7 -> 99.8 mm
- net col5: track 108.5 -> 104.6 mm
- net col1: track 174.3 -> 171.1 mm
- net col10: track 122.5 -> 125.1 mm
- net col12: track 118.7 -> 120.8 mm
- net col0: track 171.0 -> 169.2 mm
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
Commit message: no more errors
Parts:
- D41: moved to B.Cu
Routing:
- net Net-(D41-A): track 0.00 -> 11.9 mm

Commit message: pre disaster
Routing:
- net /GND: track 200.1 -> 322.4 mm, vias 4 -> 5
- net row3: vias 4 -> 6
Other:
- board size 295.9 x 87 mm -> 295.8 x 87 mm

Commit message: before disaster
Parts:
- added D52: 1N4004, ergodonk_simple_zero:D_DO-41_SOD81_P10.16mm_Horizontal, B.Cu at (167.9, -17.6)
- added J1: Conn_01x02_Socket, ergodonk_simple_zero:PinHeader_1x02_P2.54mm_Vertical, B.Cu at (143.0, -16.8)
- added J_SOL_1: Conn_01x02_Female, ergodonk_simple_zero:PinHeader_1x02_P2.54mm_Vertical, B.Cu at (134.0, -16.8)
- added Q3: TIP120, ergodonk_simple_zero:TO-220-3_Horizontal_TabDown_ergodonk_simple_zero, B.Cu at (153.0, -12.2)
- added R4: 1k, ergodonk_simple_zero:R_Axial_DIN0309_L9.0mm_D3.2mm_P12.70mm_Horizontal, B.Cu at (153.0, -28.4)

Commit message: disaster here
Parts:
- removed C1: 0.1uF, Capacitor_SMD:C_0805_2012Metric
- removed D51: D_Schottky, Diode_SMD:D_SOD-123
- removed JSOL1: Conn_01x02_MountingPin, Connector_JST:JST_SH_SM02B-SRSS-TB_1x02-1MP_P1.00mm_Horizontal
- removed Q1: Q_NMOS_GDS, Package_TO_SOT_THT:TO-220-3_Horizontal_TabDown
- removed R1: 100, Resistor_SMD:R_0805_2012Metric
- removed R2: 100k, Resistor_SMD:R_0805_2012Metric
- moved D52 135.9 mm to (191.9, 116.1)
- moved J1 135.9 mm to (167.0, 117.0)
- moved J_SOL_1 135.9 mm to (158.0, 117.0)
- moved R4 134.5 mm to (159.5, 105.9), turned to 90 degrees
- moved Q3 106.1 mm to (164.5, 93.3)
Routing:
- net /GND: track 322.4 -> 184.6 mm, vias 5 -> 3
- net /COIL_LOW: track 72.2 -> 45.9 mm
- net Net-(Q1-G): track 14.8 -> 0.00 mm
- net /+5V_SOL: track 197.3 -> 188.9 mm
- net /SOLENOID_EN: track 74.9 -> 72.5 mm
Other:
- board size 295.8 x 87 mm -> 295.5 x 84.1 mm

Commit message: rewiring time
Parts:
- removed J1: Conn_01x02_Socket, ergodonk_simple_zero:PinHeader_1x02_P2.54mm_Vertical
- removed R4: 1k, ergodonk_simple_zero:R_Axial_DIN0309_L9.0mm_D3.2mm_P12.70mm_Horizontal
- added R1: 1k, Resistor_THT:R_Axial_DIN0309_L9.0mm_D3.2mm_P12.70mm_Horizontal, B.Cu at (204.2, 148.4)
- moved D9 86.0 mm to (245.2, 114.5)
- moved D40 85.8 mm to (323.9, 152.3)
- moved D27 85.8 mm to (328.7, 133.2)
- moved D29 85.8 mm to (88.2, 152.3)
- moved D30 85.8 mm to (119.1, 152.3)
- moved D31 85.8 mm to (145.3, 152.3)
- moved D32 85.8 mm to (164.4, 152.3)
- moved D33 85.8 mm to (183.4, 152.3)
- moved D35 85.8 mm to (221.5, 152.3)
- moved D39 85.8 mm to (297.7, 152.3)
- moved D49 85.8 mm to (316.8, 171.3)
- moved S24 85.8 mm to (264.1, 130.2)
- moved S27 85.8 mm to (323.6, 130.2)
- moved S29 85.8 mm to (83.1, 149.2)
- moved S30 85.8 mm to (114.0, 149.2)
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Routing:
- net Net-(D52-A): track 0.00 -> 75.7 mm
- net /GND: track 184.6 -> 130.3 mm, vias 3 -> 2
- net /COIL_LOW: track 45.9 -> 0.00 mm, vias 1 -> 0
- net /+5V_SOL: track 188.9 -> 169.8 mm, vias 4 -> 2
- net Net-(Q3-B): track 0.00 -> 5.75 mm
- net Net-(D6-A): track 5.02 -> 9.06 mm
- net row3: track 284.6 -> 286.2 mm
- net /SOLENOID_EN: track 72.5 -> 71.4 mm, vias 2 -> 1
- added copper zone on B.Cu, net (none)
- added copper zone on F.Cu, net (none)
Other:
- board size 295.5 x 84.1 mm -> 295.5 x 83.5 mm

Commit message: donezo
Parts:
- removed D8: Diode, Diode_SMD:D_SOD-123
- moved D14 16.1 mm to (339.0, 116.2)
- moved D28 16.1 mm to (339.0, 135.1)
- moved D25 16.0 mm to (272.3, 135.2)
- moved D40 16.0 mm to (308.0, 154.2)
- moved D42 16.0 mm to (110.3, 173.3)
- moved D44 16.0 mm to (148.4, 173.3)
- moved D45 16.0 mm to (179.4, 173.3)
- moved D46 16.0 mm to (227.0, 173.3)
- moved D10 16.0 mm to (248.5, 116.2)
- moved D16 16.0 mm to (98.4, 135.2)
- moved D17 16.0 mm to (119.9, 135.2)
- moved D19 16.0 mm to (158.0, 135.2)
- moved D21 16.0 mm to (196.1, 135.2)
- moved D24 16.0 mm to (253.2, 135.2)
- moved D32 16.0 mm to (148.4, 154.2)
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Connections:
- S8 pad 2: Net-(D8-A) -> Y_KEY
- U1 pad 2: unconnected-(U1-1-Pad2) -> Y_KEY
Routing:
- net row1: track 350.7 -> 310.0 mm
- net row2: track 369.3 -> 329.1 mm
- net row0: track 392.2 -> 360.1 mm
- net row3: track 286.2 -> 258.6 mm
- net Net-(D8-A): track 13.0 -> 0.00 mm
- net Net-(D14-A): track 12.2 -> 4.78 mm
- net Net-(D28-A): track 12.1 -> 4.74 mm
- net Net-(D41-A): track 11.9 -> 4.82 mm
- net Net-(D38-A): track 11.9 -> 4.83 mm
- net Net-(D13-A): track 11.9 -> 4.83 mm
- net Net-(D12-A): track 11.9 -> 4.83 mm
- net Net-(D39-A): track 11.9 -> 4.83 mm
- net Net-(D47-A): track 11.9 -> 4.83 mm
- net Net-(D48-A): track 11.9 -> 4.83 mm
- net Net-(D32-A): track 11.9 -> 4.83 mm
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Other:
- board text added: "D23"
